File: DarlingtonDetector/DarlingtonDetector/DarlingtonDetector.kicad_sch (KiCad schematic)
At the start: 11 parts, among them Q101 MMBT2907, Q102 MMBT2907

Commit message: DarlingtonDetector.kicad_sch, Add decoupeling and bypass, add notes about sample transmission location.
Parts:
- added C103: 100nF, Capacitor_SMD:C_0603_1608Metric_Pad1.08x0.95mm_HandSolder, symbol Device:C
- added C106: 47uF 16V, Capacitor_SMD:CP_Elec_5x5.4, symbol Device:C_Polarized
- added D105: LED_T1.75_CLEAR_RED, GeneralPurposeAlarmDevicePCB:LED_5mm_Radial, symbol GPAD_SCH_LIB:LED_T1.75_CLEAR_WHITE
- added R101: 1R0, Resistor_SMD:R_0603_1608Metric_Pad0.98x0.95mm_HandSolder, symbol Device:R
- added R304: 1K, Resistor_SMD:R_0603_1608Metric_Pad0.98x0.95mm_HandSolder, symbol Device:R
Connections:
- net GND: now also C103.2, C106.2, D105.2
- net at Q102.2 (E): now also C103.1, C106.1, R101.2; no longer A101.5 (+5V)
- new net: D105.1, R304.1
- new net: A101.5 (+5V), R101.1, R304.2
Other:
- note added: "I & Q Indicators Red In phase Green Quadrature"
- note added: "Place transmission sample between Outpu and Input LEDs."
- note added: "Power Indicator"
